File: signal_driver_pcb.kicad_pcb (KiCad board)
At the start: 4 copper layers, 30 x 50 mm, 43 parts, among them J1 Conn_01x04, J2 Conn_02x03_Odd_Even, J3 Conn_02x03_Odd_Even, U1 UMCC_50Ohm, U2 UMCC_50Ohm, U3 TLV3501, U4 TLV3501, U5 DS1023, U6 NC7WZ16, U7 UMCC_50Ohm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

Commit message: committed previously uncommitted changes
Parts:
- R11: value 1k -> 2.2k
Changed lines of the file:
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@@
   (page A4)
   (layers
-    (0 F.Cu signal hide)
+    (0 F.Cu signal)
     (1 In1.Cu signal hide)
     (2 In2.Cu signal hide)
@@
     (visible_elements 7FFFFE7F)
     (pcbplotparams
-      (layerselection 0x010fc_00000000)
+      (layerselection 0x010fc_ffffffff)
       (usegerberextensions false)
       (usegerberattributes false)
@@
       (drillshape 0)
       (scaleselection 1)
-      (outputdirectory ""))
+      (outputdirectory "output/gerber_1v0/"))
   )
   (net 0 "")
@@
     (at 141.3 84.45 90)
     (attr smd)
-    (fp_text reference U5 (at 0 -6 270) (layer F.SilkS)
+    (fp_text reference U5 (at -3.95 -6.55) (layer F.SilkS)
       (effects (font (size 1 1) (thickness 0.15)))
     )
@@
       (effects (font (size 1 1) (thickness 0.15)))
     )
-    (fp_text value 1k (at 0 1.43) (layer F.Fab)
+    (fp_text value 2.2k (at 0 1.43) (layer F.Fab)
       (effects (font (size 1 1) (thickness 0.15)))
     )
@@
     (tags SOT-23-6)
     (attr smd)
-    (fp_text reference U4 (at -3.6 -3.1) (layer F.SilkS)
+    (fp_text reference U4 (at -3 -0.6) (layer F.SilkS)
       (effects (font (size 1 1) (thickness 0.15)))
     )
@@
   (segment (start 147.459808 93.295199) (end 147.588306 93.295199) (width 0.2032) (layer B.Cu) (net 6))
   (segment (start 150.392 93.75) (end 150.622 93.98) (width 0.2032) (layer B.Cu) (net 6))
-  (segment (start 128.27 97.536) (end 129.54 96.266) (width 1.016) (layer B.Cu) (net 46))
-  (segment (start 150.622 96.52) (end 151.638 97.536) (width 1.016) (layer B.Cu) (net 46))
-  (segment (start 151.765 97.536) (end 151.638 97.536) (width 1.016) (layer B.Cu) (net 46))
-  (segment (start 150.368 96.266) (end 150.622 96.52) (width 0.2032) (layer B.Cu) (net 46))
-  (segment (start 147.716 96.266) (end 150.368 96.266) (width 0.2032) (layer B.Cu) (net 46))
-  (segment (start 134.08166 93.693589) (end 145.143589 93.693589) (width 0.2032) (layer B.Cu) (net 46))
-  (segment (start 129.54 96.266) (end 131.509249 96.266) (width 0.2032) (layer B.Cu) (net 46))
-  (segment (start 131.509249 96.266) (end 134.08166 93.693589) (width 0.2032) (layer B.Cu) (net 46))
   (segment (start 128.27 105.156) (end 129.54 103.886) (width 1.016) (layer B.Cu) (net 7))
   (segment (start 150.495 103.886) (end 151.765 105.156) (width 1.016) (layer B.Cu) (net 7))
@@
   (segment (start 149.225 110.236) (end 147.952208 110.236) (width 0.2032) (layer B.Cu) (net 8))
   (segment (start 143.540243 105.824035) (end 136.239739 105.824035) (width 0.2032) (layer B.Cu) (net 8))
-  (segment (start 148.285202 98.374202) (end 148.717 98.806) (width 0.2032) (layer B.Cu) (net 44))
-  (segment (start 147.370798 98.374202) (end 148.285202 98.374202) (width 0.2032) (layer B.Cu) (net 44))
-  (segment (start 150.495 98.806) (end 148.717 98.806) (width 0.2032) (layer B.Cu) (net 44))
-  (segment (start 150.622 98.933) (end 150.495 98.806) (width 0.2032) (layer B.Cu) (net 44))
-  (segment (start 150.622 98.933) (end 151.765 100.076) (width 1.016) (layer B.Cu) (net 44))
-  (segment (start 128.27 100.076) (end 129.54 98.806) (width 1.016) (layer B.Cu) (net 44))
-  (segment (start 145.33738 100.4) (end 147.36318 98.3742) (width 0.2032) (layer B.Cu) (net 44))
-  (segment (start 129.54 98.806) (end 132.54482 98.806) (width 0.2032) (layer B.Cu) (net 44))
-  (segment (start 132.54482 98.806) (end 134.13882 100.4) (width 0.2032) (layer B.Cu) (net 44))
-  (segment (start 147.36318 98.3742) (end 147.3708 98.3742) (width 0.2032) (layer B.Cu) (net 44))
   (segment (start 128.27 102.616) (end 129.54 101.346) (width 1.016) (layer B.Cu) (net 9))
   (segment (start 150.622 101.473) (end 151.765 102.616) (width 1.016) (layer B.Cu) (net 9))
@@
   (segment (start 147.981199 83.631199) (end 147.01519 82.66519) (width 0.2032) (layer B.Cu) (net 20))
   (segment (start 147.01519 82.66519) (end 147.01519 82.05794) (width 0.2032) (layer B.Cu) (net 20))
-  (segment (start 130.81 97.536) (end 131.826 97.536) (width 1.016) (layer B.Cu) (net 45))
-  (segment (start 147.828 97.536) (end 149.225 97.536) (width 1.016) (layer B.Cu) (net 45))
-  (segment (start 147.586 97.536) (end 147.828 97.536) (width 0.2032) (layer B.Cu) (net 45))
-  (segment (start 144.15 94.1) (end 147.586 97.536) (width 0.2032) (layer B.Cu) (net 45))
-  (segment (start 131.826 97.536) (end 131.826 96.524) (width 0.2032) (layer B.Cu) (net 45))
-  (segment (start 131.826 96.524) (end 134.25 94.1) (width 0.2032) (layer B.Cu) (net 45))
   (segment (start 130.81 105.156) (end 131.826 105.156) (width 1.016) (layer B.Cu) (net 21))
   (segment (start 148.463 105.156) (end 149.225 105.156) (width 1.016) (layer B.Cu) (net 21))
@@
   (segment (start 136.054802 98.295198) (end 137.74031 98.295198) (width 0.2032) (layer F.Cu) (net 43))
   (segment (start 136.05 98.3) (end 136.054802 98.295198) (width 0.2032) (layer F.Cu) (net 43))
+  (segment (start 148.285202 98.374202) (end 148.717 98.806) (width 0.2032) (layer B.Cu) (net 44))
+  (segment (start 147.370798 98.374202) (end 148.285202 98.374202) (width 0.2032) (layer B.Cu) (net 44))
+  (segment (start 150.495 98.806) (end 148.717 98.806) (width 0.2032) (layer B.Cu) (net 44))
+  (segment (start 150.622 98.933) (end 150.495 98.806) (width 0.2032) (layer B.Cu) (net 44))
+  (segment (start 150.622 98.933) (end 151.765 100.076) (width 1.016) (layer B.Cu) (net 44))
+  (segment (start 128.27 100.076) (end 129.54 98.806) (width 1.016) (layer B.Cu) (net 44))
+  (segment (start 145.33738 100.4) (end 147.36318 98.3742) (width 0.2032) (layer B.Cu) (net 44))
+  (segment (start 129.54 98.806) (end 132.54482 98.806) (width 0.2032) (layer B.Cu) (net 44))
+  (segment (start 132.54482 98.806) (end 134.13882 100.4) (width 0.2032) (layer B.Cu) (net 44))
+  (segment (start 147.36318 98.3742) (end 147.3708 98.3742) (width 0.2032) (layer B.Cu) (net 44))
   (segment (start 136.845193 96.429807) (end 137.30429 95.97071) (width 0.2032) (layer B.Cu) (net 44))
   (segment (start 136.845193 99.190305) (end 136.845193 96.429807) (width 0.2032) (layer B.Cu) (net 44))
@@
   (segment (start 137.05 100.4) (end 145.33738 100.4) (width 0.2032) (layer B.Cu) (net 44))
   (segment (start 134.13882 100.4) (end 137.05 100.4) (width 0.2032) (layer B.Cu) (net 44))
+  (segment (start 130.81 97.536) (end 131.826 97.536) (width 1.016) (layer B.Cu) (net 45))
+  (segment (start 147.828 97.536) (end 149.225 97.536) (width 1.016) (layer B.Cu) (net 45))
+  (segment (start 147.586 97.536) (end 147.828 97.536) (width 0.2032) (layer B.Cu) (net 45))
+  (segment (start 144.15 94.1) (end 147.586 97.536) (width 0.2032) (layer B.Cu) (net 45))
+  (segment (start 131.826 97.536) (end 131.826 96.524) (width 0.2032) (layer B.Cu) (net 45))
+  (segment (start 131.826 96.524) (end 134.25 94.1) (width 0.2032) (layer B.Cu) (net 45))
   (segment (start 139.025 94.175) (end 138.95 94.1) (width 0.2032) (layer B.Cu) (net 45))
   (segment (start 139.025 95.5) (end 139.025 94.175) (width 0.2032) (layer B.Cu) (net 45))
   (segment (start 134.25 94.1) (end 138.95 94.1) (width 0.2032) (layer B.Cu) (net 45))
   (segment (start 138.95 94.1) (end 144.15 94.1) (width 0.2032) (layer B.Cu) (net 45))
+  (segment (start 128.27 97.536) (end 129.54 96.266) (width 1.016) (layer B.Cu) (net 46))
+  (segment (start 150.622 96.52) (end 151.638 97.536) (width 1.016) (layer B.Cu) (net 46))
+  (segment (start 151.765 97.536) (end 151.638 97.536) (width 1.016) (layer B.Cu) (net 46))
+  (segment (start 150.368 96.266) (end 150.622 96.52) (width 0.2032) (layer B.Cu) (net 46))
+  (segment (start 147.716 96.266) (end 150.368 96.266) (width 0.2032) (layer B.Cu) (net 46))
+  (segment (start 134.08166 93.693589) (end 145.143589 93.693589) (width 0.2032) (layer B.Cu) (net 46))
+  (segment (start 129.54 96.266) (end 131.509249 96.266) (width 0.2032) (layer B.Cu) (net 46))
+  (segment (start 131.509249 96.266) (end 134.08166 93.693589) (width 0.2032) (layer B.Cu) (net 46))
   (via (at 147.077659 96.172341) (size 0.6) (drill 0.4) (layers F.Cu B.Cu) (net 46))
   (segment (start 147.25 96) (end 147.077659 96.172341) (width 0.2032) (layer B.Cu) (net 46))
